Commit message: fix(urdf): rename joint join3 to joint3 Aligns the default SDK URDF with ROS bringup and arm.yaml naming.
(cherry picked from commit 2828b64096c70ad46ff0af3d74e8110d278abaa3)

File: urdf/reBot-DevArm_fixend_description/urdf/reBot-DevArm_fixend.urdf (robot description, URDF)
Before this commit: robot reBot-DevArm_fixend, 8 links, 7 joints
Joints:
- removed joint join3
- added joint joint3: type revolute, parent link2, child link3, origin xyz=-0.264 0 0 rpy=0 0 0, axis 0 0 1, limit lower=-3.14 upper=0 effort=27 velocity=50
